Commit message: fix(foot_quadruped): give VbotBaboEDU head joints real servo limits
The head_yaw_joint and head_pitch_joint limits were effort="0"
velocity="0". Simulators read that two ways: some apply no torque, so
the head drops onto its stop, and others treat it as unlimited. Both
URDFs now use the head servo spec: stall torque 30 kgf·cm ≈ 2.94 N·m
and a 0.5 rad/s velocity cap enforced by the control code.

In the mock_head variants, the head inertia is now scaled by the ratio
of mock mass to real mass. The links had kept the full head's inertia
on 1e-8 / 1e-6 kg masses, which gave a radius of gyration of about
600 m.

Synced from vitamin VitaDynamics/vitamin#70.

Co-Authored-By: Claude Opus 5.5 <noreply@anthropic.com>

File: assets/robots/foot_quadruped/urdf/VbotBaboEDU.urdf (robot description, URDF)
Before this commit: robot VbotBaboEDU, 20 links, 19 joints
Joints:
- joint head_pitch_joint: limit lower=-0.5236 upper=0.20944 effort=0 velocity=0 -> lower=-0.5236 upper=0.20944 effort=2.94 velocity=0.5
- joint head_yaw_joint: limit lower=-0.69813 upper=0.69813 effort=0 velocity=0 -> lower=-0.69813 upper=0.69813 effort=2.94 velocity=0.5

File: assets/robots/foot_quadruped/urdf/VbotBaboEDU_backboard.urdf (robot description, URDF)
Before this commit: robot VbotBaboEDU, 21 links, 20 joints
Joints:
- joint head_pitch_joint: limit lower=-0.5236 upper=0.20944 effort=0 velocity=0 -> lower=-0.5236 upper=0.20944 effort=2.94 velocity=0.5
- joint head_yaw_joint: limit lower=-0.69813 upper=0.69813 effort=0 velocity=0 -> lower=-0.69813 upper=0.69813 effort=2.94 velocity=0.5

File: assets/robots/foot_quadruped/urdf/VbotBaboEDU_backboard_bracket.urdf (robot description, URDF)
Before this commit: robot VbotBaboEDU, 22 links, 21 joints
Joints:
- joint head_pitch_joint: limit lower=-0.5236 upper=0.20944 effort=0 velocity=0 -> lower=-0.5236 upper=0.20944 effort=2.94 velocity=0.5
- joint head_yaw_joint: limit lower=-0.69813 upper=0.69813 effort=0 velocity=0 -> lower=-0.69813 upper=0.69813 effort=2.94 velocity=0.5

File: assets/robots/foot_quadruped/urdf/VbotBaboEDU_mock_head.urdf (robot description, URDF)
Before this commit: robot VbotBaboEDU, 20 links, 19 joints
Joints:
- joint head_pitch_joint: limit lower=-0.5236 upper=0.20944 effort=0 velocity=0 -> lower=-0.5236 upper=0.20944 effort=2.94 velocity=0.5
- joint head_yaw_joint: limit lower=-0.69813 upper=0.69813 effort=0 velocity=0 -> lower=-0.69813 upper=0.69813 effort=2.94 velocity=0.5

File: assets/robots/foot_quadruped/urdf/VbotBaboEDU_mock_head_silence.urdf (robot description, URDF)
Before this commit: robot VbotBaboEDU, 20 links, 19 joints
Joints:
- joint head_pitch_joint: limit lower=-0.5236 upper=0.20944 effort=0 velocity=0 -> lower=-0.5236 upper=0.20944 effort=2.94 velocity=0.5
- joint head_yaw_joint: limit lower=-0.69813 upper=0.69813 effort=0 velocity=0 -> lower=-0.69813 upper=0.69813 effort=2.94 velocity=0.5
